File: pcb_schematic/touchpad.kicad_pcb (KiCad board)
At the start: 2 copper layers, 119.4 x 62 mm, 12 parts, among them U1 touchpad, U2 CD74HC4067M, U3 ProMicro

Commit message: Update PCB
Connections:
- net /SIG3 renamed /S0
- U2 pad 11: /SIG2 -> /S1
- U2 pad 13: /SIG1 -> /S3
- U2 pad 14: /SIG0 -> /S2
- U3 pad 14: /SIG0 -> /S1
- U3 pad 15: /SIG1 -> /S2
- U3 pad 16: unconnected-(U3-Pad16) -> /S3
- U3 pad 6: PWM -> unconnected-(U3-Pad6)
- U3 pad 8: /SIG2 -> PWM
Routing:
- net /S1: track 0.00 -> 39.0 mm
- net /SIG0: track 37.2 -> 0.00 mm
- net /S2: track 0.00 -> 35.1 mm
- net /SIG1: track 32.8 -> 0.00 mm
- net /S3: track 0.00 -> 31.4 mm
- net /SIG2: track 29.2 -> 0.00 mm
- net PWM: track 44.5 -> 49.5 mm
- net /S0: track 36.0 -> 38.6 mm
Changed lines of the file:
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@@
   (net 10 "/ADC10")
   (net 11 "PWM")
-  (net 12 "/SIG0")
-  (net 13 "/SIG1")
-  (net 14 "/SIG3")
-  (net 15 "/SIG2")
+  (net 12 "/S0")
+  (net 13 "/S1")
+  (net 14 "/S3")
+  (net 15 "/S2")
   (net 16 "/Vcc")
   (net 17 "unconnected-(U3-Pad1)")
@@
   (net 36 "Net-(U1-PadTx15)")
   (net 37 "Net-(U1-PadTx16)")
-  (net 38 "unconnected-(U3-Pad16)")
+  (net 38 "unconnected-(U3-Pad6)")
   (footprint "promicro:ProMicro" placed (layer "F.Cu")
     (at 88.9 83.82 -90)
@@
       (net 19 "unconnected-(U3-Pad5)") (pinfunction "SDA") (pintype "bidirectional"))
     (pad "6" thru_hole circle locked (at -1.27 7.62 270) (size 1.6 1.6) (drill 1.1) (layers *.Cu *.Mask "F.SilkS")
-      (net 11 "PWM") (pinfunction "SCL") (pintype "bidirectional"))
+      (net 38 "unconnected-(U3-Pad6)") (pinfunction "SCL") (pintype "bidirectional"))
     (pad "7" thru_hole circle locked (at 1.27 7.62 270) (size 1.6 1.6) (drill 1.1) (layers *.Cu *.Mask "F.SilkS")
       (net 6 "/ADC6") (pinfunction "D4") (pintype "bidirectional"))
     (pad "8" thru_hole circle locked (at 3.81 7.62 270) (size 1.6 1.6) (drill 1.1) (layers *.Cu *.Mask "F.SilkS")
-      (net 15 "/SIG2") (pinfunction "C6") (pintype "bidirectional"))
+      (net 11 "PWM") (pinfunction "C6") (pintype "bidirectional"))
     (pad "9" thru_hole circle locked (at 6.35 7.62 270) (size 1.6 1.6) (drill 1.1) (layers *.Cu *.Mask "F.SilkS")
       (net 7 "/ADC7") (pinfunction "D7") (pintype "bidirectional"))
     (pad "10" thru_hole circle locked (at 8.89 7.62 270) (size 1.6 1.6) (drill 1.1) (layers *.Cu *.Mask "F.SilkS")
-      (net 14 "/SIG3") (pinfunction "E6") (pintype "bidirectional"))
+      (net 12 "/S0") (pinfunction "E6") (pintype "bidirectional"))
     (pad "11" thru_hole circle locked (at 11.43 7.62 270) (size 1.6 1.6) (drill 1.1) (layers *.Cu *.Mask "F.SilkS")
       (net 8 "/ADC8") (pinfunction "B4") (pintype "bidirectional"))
@@
       (net 10 "/ADC10") (pinfunction "B6") (pintype "bidirectional"))
     (pad "14" thru_hole circle locked (at 11.43 -7.62 270) (size 1.6 1.6) (drill 1.1) (layers *.Cu *.Mask "F.SilkS")
-      (net 12 "/SIG0") (pinfunction "B2") (pintype "bidirectional"))
+      (net 13 "/S1") (pinfunction "B2") (pintype "bidirectional"))
     (pad "15" thru_hole circle locked (at 8.89 -7.62 270) (size 1.6 1.6) (drill 1.1) (layers *.Cu *.Mask "F.SilkS")
-      (net 13 "/SIG1") (pinfunction "B3") (pintype "bidirectional"))
+      (net 15 "/S2") (pinfunction "B3") (pintype "bidirectional"))
     (pad "16" thru_hole circle locked (at 6.35 -7.62 270) (size 1.6 1.6) (drill 1.1) (layers *.Cu *.Mask "F.SilkS")
-      (net 38 "unconnected-(U3-Pad16)") (pinfunction "B1") (pintype "bidirectional"))
+      (net 14 "/S3") (pinfunction "B1") (pintype "bidirectional"))
     (pad "17" thru_hole circle locked (at 3.81 -7.62 270) (size 1.6 1.6) (drill 1.1) (layers *.Cu *.Mask "F.SilkS")
       (net 2 "/ADC0") (pinfunction "F7") (pintype "bidirectional"))
@@
       (net 37 "Net-(U1-PadTx16)") (pinfunction "I0") (pintype "passive"))
     (pad "10" smd roundrect (at -4.65 4.445) (size 2.05 0.6) (layers "F.Cu" "F.Paste" "F.Mask") (roundrect_rratio 0.25)
-      (net 14 "/SIG3") (pinfunction "S0") (pintype "input"))
+      (net 12 "/S0") (pinfunction "S0") (pintype "input"))
     (pad "11" smd roundrect (at -4.65 5.715) (size 2.05 0.6) (layers "F.Cu" "F.Paste" "F.Mask") (roundrect_rratio 0.25)
-      (net 15 "/SIG2") (pinfunction "S1") (pintype "input"))
+      (net 13 "/S1") (pinfunction "S1") (pintype "input"))
     (pad "12" smd roundrect (at -4.65 6.985) (size 2.05 0.6) (layers "F.Cu" "F.Paste" "F.Mask") (roundrect_rratio 0.25)
       (net 1 "/GND") (pinfunction "GND") (pintype "power_in"))
     (pad "13" smd roundrect (at 4.65 6.985) (size 2.05 0.6) (layers "F.Cu" "F.Paste" "F.Mask") (roundrect_rratio 0.25)
-      (net 13 "/SIG1") (pinfunction "S3") (pintype "input"))
+      (net 14 "/S3") (pinfunction "S3") (pintype "input"))
     (pad "14" smd roundrect (at 4.65 5.715) (size 2.05 0.6) (layers "F.Cu" "F.Paste" "F.Mask") (roundrect_rratio 0.25)
-      (net 12 "/SIG0") (pinfunction "S2") (pintype "input"))
+      (net 15 "/S2") (pinfunction "S2") (pintype "input"))
     (pad "15" smd roundrect (at 4.65 4.445) (size 2.05 0.6) (layers "F.Cu" "F.Paste" "F.Mask") (roundrect_rratio 0.25)
       (net 1 "/GND") (pinfunction "~{E}") (pintype "input"))
@@
   (segment (start 84.885 48.26) (end 88.9 48.26) (width 0.25) (layer "F.Cu") (net 11))
   (segment (start 84.25 48.895) (end 84.885 48.26) (width 0.25) (layer "F.Cu") (net 11))
-  (via blind (at 88.9 48.26) (size 0.8) (drill 0.4) (layers "F.Cu" "B.Cu") (net 11))
-  (segment (start 78.74 80.01) (end 78.74 58.42) (width 0.25) (layer "B.Cu") (net 11))
-  (segment (start 78.74 58.42) (end 88.9 48.26) (width 0.25) (layer "B.Cu") (net 11))
-  (segment (start 81.28 82.55) (end 78.74 80.01) (width 0.25) (layer "B.Cu") (net 11))
-  (segment (start 93.976751 61.595) (end 99.06 66.678249) (width 0.25) (layer "F.Cu") (net 12))
-  (segment (start 99.06 92.71) (end 96.52 95.25) (width 0.25) (layer "F.Cu") (net 12))
-  (segment (start 99.06 66.678249) (end 99.06 92.71) (width 0.25) (layer "F.Cu") (net 12))
-  (segment (start 93.55 61.595) (end 93.976751 61.595) (width 0.25) (layer "F.Cu") (net 12))
-  (segment (start 98.61 90.62) (end 96.52 92.71) (width 0.25) (layer "F.Cu") (net 13))
-  (segment (start 98.61 67.925) (end 98.61 90.62) (width 0.25) (layer "F.Cu") (net 13))
-  (segment (start 93.55 62.865) (end 98.61 67.925) (width 0.25) (layer "F.Cu") (net 13))
-  (segment (start 78.74 65.408249) (end 78.74 90.17) (width 0.25) (layer "F.Cu") (net 14))
-  (segment (start 84.25 60.325) (end 83.823249 60.325) (width 0.25) (layer "F.Cu") (net 14))
-  (segment (start 78.74 90.17) (end 81.28 92.71) (width 0.25) (layer "F.Cu") (net 14))
-  (segment (start 83.823249 60.325) (end 78.74 65.408249) (width 0.25) (layer "F.Cu") (net 14))
-  (segment (start 79.19 66.228249) (end 79.19 85.54) (width 0.25) (layer "F.Cu") (net 15))
-  (segment (start 83.823249 61.595) (end 79.19 66.228249) (width 0.25) (layer "F.Cu") (net 15))
-  (segment (start 79.19 85.54) (end 81.28 87.63) (width 0.25) (layer "F.Cu") (net 15))
-  (segment (start 84.25 61.595) (end 83.823249 61.595) (width 0.25) (layer "F.Cu") (net 15))
+  (via (at 88.9 48.26) (size 0.8) (drill 0.4) (layers "F.Cu" "B.Cu") (net 11))
+  (segment (start 78.74 58.42) (end 78.74 85.09) (width 0.25) (layer "B.Cu") (net 11))
+  (segment (start 88.9 48.26) (end 78.74 58.42) (width 0.25) (layer "B.Cu") (net 11))
+  (segment (start 78.74 85.09) (end 81.28 87.63) (width 0.25) (layer "B.Cu") (net 11))
+  (segment (start 78.74 90.17) (end 81.28 92.71) (width 0.25) (layer "F.Cu") (net 12))
+  (segment (start 84.25 60.325) (end 79.375 60.325) (width 0.25) (layer "F.Cu") (net 12))
+  (segment (start 78.74 60.96) (end 78.74 90.17) (width 0.25) (layer "F.Cu") (net 12))
+  (segment (start 79.375 60.325) (end 78.74 60.96) (width 0.25) (layer "F.Cu") (net 12))
+  (segment (start 84.676751 61.595) (end 86.36 63.278249) (width 0.25) (layer "F.Cu") (net 13))
+  (segment (start 84.25 61.595) (end 84.676751 61.595) (width 0.25) (layer "F.Cu") (net 13))
+  (segment (start 86.36 85.09) (end 96.52 95.25) (width 0.25) (layer "F.Cu") (net 13))
+  (segment (start 86.36 63.278249) (end 86.36 85.09) (width 0.25) (layer "F.Cu") (net 13))
+  (segment (start 96.52 90.17) (end 97.79 90.17) (width 0.25) (layer "F.Cu") (net 14))
+  (segment (start 99.06 88.9) (end 99.06 68.375) (width 0.25) (layer "F.Cu") (net 14))
+  (segment (start 97.79 90.17) (end 99.06 88.9) (width 0.25) (layer "F.Cu") (net 14))
+  (segment (start 99.06 68.375) (end 93.55 62.865) (width 0.25) (layer "F.Cu") (net 14))
+  (segment (start 99.509501 89.720499) (end 99.509501 67.12775) (width 0.25) (layer "F.Cu") (net 15))
+  (segment (start 93.976751 61.595) (end 93.55 61.595) (width 0.25) (layer "F.Cu") (net 15))
+  (segment (start 96.52 92.71) (end 99.509501 89.720499) (width 0.25) (layer "F.Cu") (net 15))
+  (segment (start 99.509501 67.12775) (end 93.976751 61.595) (width 0.25) (layer "F.Cu") (net 15))
   (segment (start 88.9 53.118249) (end 88.9 69.85) (width 0.25) (layer "F.Cu") (net 16))
   (segment (start 93.123249 48.895) (end 88.9 53.118249) (width 0.25) (layer "F.Cu") (net 16))
